File: Robot_Veloz-master/Robot_Veloz-master/Robot_Veloz-master/Robot_Veloz/Robot_Veloz/Hardware/Placa/Placa/Placa.sch (KiCad schematic (older format))
At the start: 39 parts, among them J1 Conn_01x03, J10 Conn_01x03, J11 Conn_01x03, J12 Conn_01x03, J13 Conn_01x02, J14 Conn_01x02, J15 Conn_01x08, J16 Conn_01x08, J2 Conn_01x03, J3 Conn_01x03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

Commit message: esquema placa terminado
Parts:
- J1, J10, J11, J12, J2, J4, J5: footprint Connector_PinHeader_2.54mm:PinHeader_1x06_P2.54mm_Vertical -> Connector_PinHeader_2.54mm:PinHeader_1x03_P2.54mm_Vertical
- J13, J14: footprint Connector_PinHeader_2.54mm:PinHeader_1x06_P2.54mm_Vertical -> Connector_PinHeader_2.54mm:PinHeader_1x02_P2.54mm_Vertical
- J15, J16: footprint Connector_PinHeader_2.54mm:PinHeader_1x06_P2.54mm_Vertical -> Connector_PinHeader_2.54mm:PinHeader_1x08_P2.54mm_Vertical
- J3: footprint Connector_JST:JST_XH_B03B-XH-A_1x03_P2.50mm_Vertical -> Connector_PinHeader_2.54mm:PinHeader_1x03_P2.54mm_Vertical
- J6, J7: footprint Connector_JST:JST_XH_B03B-XH-A_1x03_P2.50mm_Vertical -> Connector_PinHeader_2.54mm:PinHeader_1x02_P2.54mm_Vertical
- JP1: footprint (none) -> Jumper:SolderJumper-3_P1.3mm_Open_Pad1.0x1.5mm
- SW1, SW2: footprint (none) -> Button_Switch_THT:SW_PUSH_6mm
- SW3: footprint (none) -> Button_Switch_THT:SW_CuK_JS202011CQN_DPDT_Straight
- U1: footprint (none) -> Package_DIP:DIP-16_W7.62mm_LongPads
- U2: footprint (none) -> Placa:DC-DC-MP2307
Changed lines of the file:
@@
 F 0 "SW1" H 2150 1885 50  0000 C CNN
 F 1 "SW_Push" H 2150 1794 50  0000 C CNN
-F 2 "" H 2150 1800 50  0001 C CNN
+F 2 "Button_Switch_THT:SW_PUSH_6mm" H 2150 1800 50  0001 C CNN
 F 3 "" H 2150 1800 50  0001 C CNN
 	1    2150 1600
@@
 F 0 "SW2" H 2600 1885 50  0000 C CNN
 F 1 "SW_Push" H 2600 1794 50  0000 C CNN
-F 2 "" H 2600 1800 50  0001 C CNN
+F 2 "Button_Switch_THT:SW_PUSH_6mm" H 2600 1800 50  0001 C CNN
 F 3 "" H 2600 1800 50  0001 C CNN
 	1    2600 1600
@@
 F 0 "J3" H 720 2625 50  0000 C CNN
 F 1 "Conn_01x03" H 720 2716 50  0000 C CNN
-F 2 "Connector_JST:JST_XH_B03B-XH-A_1x03_P2.50mm_Vertical" H 800 2950 50  0001 C CNN
+F 2 "Connector_PinHeader_2.54mm:PinHeader_1x03_P2.54mm_Vertical" H 800 2950 50  0001 C CNN
 F 3 "~" H 800 2950 50  0001 C CNN
 	1    800  2950
@@
 F 0 "J6" H 1620 2375 50  0000 C CNN
 F 1 "Conn_01x02" H 1620 2466 50  0000 C CNN
-F 2 "Connector_JST:JST_XH_B03B-XH-A_1x03_P2.50mm_Vertical" H 1700 2700 50  0001 C CNN
+F 2 "Connector_PinHeader_2.54mm:PinHeader_1x02_P2.54mm_Vertical" H 1700 2700 50  0001 C CNN
 F 3 "~" H 1700 2700 50  0001 C CNN
 	1    1700 2700
@@
 F 0 "J7" H 1620 2775 50  0000 C CNN
 F 1 "Conn_01x02" H 1620 2866 50  0000 C CNN
-F 2 "Connector_JST:JST_XH_B03B-XH-A_1x03_P2.50mm_Vertical" H 1700 3100 50  0001 C CNN
+F 2 "Connector_PinHeader_2.54mm:PinHeader_1x02_P2.54mm_Vertical" H 1700 3100 50  0001 C CNN
 F 3 "~" H 1700 3100 50  0001 C CNN
 	1    1700 3100
@@
 F 0 "J1" H 620 4225 50  0000 C CNN
 F 1 "Conn_01x03" H 620 4316 50  0000 C CNN
-F 2 "Connector_PinHeader_2.54mm:PinHeader_1x06_P2.54mm_Vertical" H 700 4550 50  0001 C CNN
+F 2 "Connector_PinHeader_2.54mm:PinHeader_1x03_P2.54mm_Vertical" H 700 4550 50  0001 C CNN
 F 3 "~" H 700 4550 50  0001 C CNN
 	1    700  4550
@@
 F 0 "J2" H 620 4775 50  0000 C CNN
 F 1 "Conn_01x03" H 620 4866 50  0000 C CNN
-F 2 "Connector_PinHeader_2.54mm:PinHeader_1x06_P2.54mm_Vertical" H 700 5100 50  0001 C CNN
+F 2 "Connector_PinHeader_2.54mm:PinHeader_1x03_P2.54mm_Vertical" H 700 5100 50  0001 C CNN
 F 3 "~" H 700 5100 50  0001 C CNN
 	1    700  5100
@@
 F 0 "J4" H 1470 4225 50  0000 C CNN
 F 1 "Conn_01x03" H 1470 4316 50  0000 C CNN
-F 2 "Connector_PinHeader_2.54mm:PinHeader_1x06_P2.54mm_Vertical" H 1550 4550 50  0001 C CNN
+F 2 "Connector_PinHeader_2.54mm:PinHeader_1x03_P2.54mm_Vertical" H 1550 4550 50  0001 C CNN
 F 3 "~" H 1550 4550 50  0001 C CNN
 	1    1550 4550
@@
 F 0 "J5" H 1470 4775 50  0000 C CNN
 F 1 "Conn_01x03" H 1470 4866 50  0000 C CNN
-F 2 "Connector_PinHeader_2.54mm:PinHeader_1x06_P2.54mm_Vertical" H 1550 5100 50  0001 C CNN
+F 2 "Connector_PinHeader_2.54mm:PinHeader_1x03_P2.54mm_Vertical" H 1550 5100 50  0001 C CNN
 F 3 "~" H 1550 5100 50  0001 C CNN
 	1    1550 5100
@@
 F 0 "J12" H 4170 3525 50  0000 C CNN
 F 1 "Conn_01x03" H 4170 3616 50  0000 C CNN
-F 2 "Connector_PinHeader_2.54mm:PinHeader_1x06_P2.54mm_Vertical" H 4250 3850 50  0001 C CNN
+F 2 "Connector_PinHeader_2.54mm:PinHeader_1x03_P2.54mm_Vertical" H 4250 3850 50  0001 C CNN
 F 3 "~" H 4250 3850 50  0001 C CNN
 	1    4250 3850
@@
 F 0 "J11" H 4170 2475 50  0000 C CNN
 F 1 "Conn_01x03" H 4170 2566 50  0000 C CNN
-F 2 "Connector_PinHeader_2.54mm:PinHeader_1x06_P2.54mm_Vertical" H 4250 2800 50  0001 C CNN
+F 2 "Connector_PinHeader_2.54mm:PinHeader_1x03_P2.54mm_Vertical" H 4250 2800 50  0001 C CNN
 F 3 "~" H 4250 2800 50  0001 C CNN
 	1    4250 2800
@@
 F 0 "J10" H 4170 1325 50  0000 C CNN
 F 1 "Conn_01x03" H 4170 1416 50  0000 C CNN
-F 2 "Connector_PinHeader_2.54mm:PinHeader_1x06_P2.54mm_Vertical" H 4250 1650 50  0001 C CNN
+F 2 "Connector_PinHeader_2.54mm:PinHeader_1x03_P2.54mm_Vertical" H 4250 1650 50  0001 C CNN
 F 3 "~" H 4250 1650 50  0001 C CNN
 	1    4250 1650
@@
 F 0 "U1" H 6100 2928 50  0000 C CNN
 F 1 "PCF8574" H 6100 2837 50  0000 C CNN
-F 2 "" H 6100 2050 50  0001 C CNN
+F 2 "Package_DIP:DIP-16_W7.62mm_LongPads" H 6100 2050 50  0001 C CNN
 F 3 "http://www.nxp.com/documents/data_sheet/PCF8574_PCF8574A.pdf" H 6100 2050 50  0001 C CNN
 	1    6100 2050
@@
 	-1   0    0    1
 $EndComp
-$Comp
-L DC-DC_MP2307:DC-DC_BuckModule U2
-U 1 1 5C13D8E2
-P 9750 1500
-F 0 "U2" H 9750 1801 39  0000 C CNN
-F 1 "DC-DC_BuckModule" H 9750 1726 39  0000 C CNN
-F 2 "" H 9750 1500 39  0001 C CNN
-F 3 "" H 9750 1500 39  0001 C CNN
-	1    9750 1500
-	1    0    0    -1
-$EndComp
 Wire Wire Line
 	10050 1400 10150 1400
@@
 F 0 "JP1" H 9300 2535 50  0000 C CNN
 F 1 "Jumper_NO_Small" H 9300 2444 50  0000 C CNN
-F 2 "" H 9300 2350 50  0001 C CNN
+F 2 "Jumper:SolderJumper-3_P1.3mm_Open_Pad1.0x1.5mm" H 9300 2350 50  0001 C CNN
 F 3 "~" H 9300 2350 50  0001 C CNN
 	1    9300 2350
@@
 F 0 "SW3" H 7750 2735 50  0000 C CNN
 F 1 "SW_DPDT_x2" H 7750 2644 50  0000 C CNN
-F 2 "" H 7750 2450 50  0001 C CNN
+F 2 "Button_Switch_THT:SW_CuK_JS202011CQN_DPDT_Straight" H 7750 2450 50  0001 C CNN
 F 3 "" H 7750 2450 50  0001 C CNN
 	2    7750 2450
@@
 F 0 "SW3" H 7800 1585 50  0000 C CNN
 F 1 "SW_DPDT_x2" H 7800 1494 50  0000 C CNN
-F 2 "" H 7800 1300 50  0001 C CNN
+F 2 "Button_Switch_THT:SW_CuK_JS202011CQN_DPDT_Straight" H 7800 1300 50  0001 C CNN
 F 3 "" H 7800 1300 50  0001 C CNN
 	1    7800 1300
 	1    0    0    -1
 $EndComp
-Wire Wire Line
-	9450 1400 8000 1400
 NoConn ~ 7950 2350
 Text GLabel 7350 1150 1    50   Input ~ 0
@@
 F 0 "J15" H 7180 4092 50  0000 L CNN
 F 1 "Conn_01x08" H 7180 4001 50  0000 L CNN
-F 2 "Connector_PinHeader_2.54mm:PinHeader_1x06_P2.54mm_Vertical" H 7100 4100 50  0001 C CNN
+F 2 "Connector_PinHeader_2.54mm:PinHeader_1x08_P2.54mm_Vertical" H 7100 4100 50  0001 C CNN
 F 3 "~" H 7100 4100 50  0001 C CNN
 	1    7100 4100
@@
 F 0 "J16" H 7880 4092 50  0000 L CNN
 F 1 "Conn_01x08" H 7880 4001 50  0000 L CNN
-F 2 "Connector_PinHeader_2.54mm:PinHeader_1x06_P2.54mm_Vertical" H 7800 4100 50  0001 C CNN
+F 2 "Connector_PinHeader_2.54mm:PinHeader_1x08_P2.54mm_Vertical" H 7800 4100 50  0001 C CNN
 F 3 "~" H 7800 4100 50  0001 C CNN
 	1    7800 4100
@@
 F 0 "J13" H 6980 5192 50  0000 L CNN
 F 1 "Conn_01x02" H 6980 5101 50  0000 L CNN
-F 2 "Connector_PinHeader_2.54mm:PinHeader_1x06_P2.54mm_Vertical" H 6900 5200 50  0001 C CNN
+F 2 "Connector_PinHeader_2.54mm:PinHeader_1x02_P2.54mm_Vertical" H 6900 5200 50  0001 C CNN
 F 3 "~" H 6900 5200 50  0001 C CNN
 	1    6900 5200
@@
 F 0 "J14" H 6980 5542 50  0000 L CNN
 F 1 "Conn_01x02" H 6980 5451 50  0000 L CNN
-F 2 "Connector_PinHeader_2.54mm:PinHeader_1x06_P2.54mm_Vertical" H 6900 5550 50  0001 C CNN
+F 2 "Connector_PinHeader_2.54mm:PinHeader_1x02_P2.54mm_Vertical" H 6900 5550 50  0001 C CNN
 F 3 "~" H 6900 5550 50  0001 C CNN
 	1    6900 5550
@@
 Wire Wire Line
 	6650 5200 6700 5200
+Wire Wire Line
+	9450 1400 8000 1400
+$Comp
+L DC-DC_MP2307:DC-DC_BuckModule U2
+U 1 1 5C1765C0
+P 9750 1500
+F 0 "U2" H 9750 1801 39  0000 C CNN
+F 1 "DC-DC_BuckModule" H 9750 1726 39  0000 C CNN
+F 2 "Placa:DC-DC-MP2307" H 9750 1500 39  0001 C CNN
+F 3 "" H 9750 1500 39  0001 C CNN
+	1    9750 1500
+	1    0    0    -1
+$EndComp
 $EndSCHEMATC
