File: Robot_Veloz-master/Robot_Veloz-master/Robot_Veloz/Robot_Veloz/Hardware/Placa/Placa/Placa.sch (KiCad schematic (older format))
At the start: 39 parts, among them J1 Conn_01x03, J10 Conn_01x03, J11 Conn_01x03, J12 Conn_01x03, J13 Conn_01x02, J14 Conn_01x02, J15 Conn_01x08, J16 Conn_01x08, J2 Conn_01x03, J3 Conn_01x03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

Commit message: esquema placa terminado
Parts:
- JP1: footprint Jumper:SolderJumper-3_P1.3mm_Open_Pad1.0x1.5mm -> (none)
- SW1, SW2: footprint Buttons_Switches_THT:SW_PUSH_6mm -> (none)
- SW3: footprint Buttons_Switches_THT:SW_CuK_JS202011CQN_DPDT_Straight -> (none)
- U1: footprint Housings_DIP:DIP-16_W7.62mm_LongPads -> (none)
- U2: footprint Placa:DC-DC-MP2307 -> (none)
Changed lines of the file:
@@
 F 0 "SW1" H 2150 1885 50  0000 C CNN
 F 1 "SW_Push" H 2150 1794 50  0000 C CNN
-F 2 "Buttons_Switches_THT:SW_PUSH_6mm" H 2150 1800 50  0001 C CNN
+F 2 "" H 2150 1800 50  0001 C CNN
 F 3 "" H 2150 1800 50  0001 C CNN
 	1    2150 1600
@@
 F 0 "SW2" H 2600 1885 50  0000 C CNN
 F 1 "SW_Push" H 2600 1794 50  0000 C CNN
-F 2 "Buttons_Switches_THT:SW_PUSH_6mm" H 2600 1800 50  0001 C CNN
+F 2 "" H 2600 1800 50  0001 C CNN
 F 3 "" H 2600 1800 50  0001 C CNN
 	1    2600 1600
@@
 F 0 "U1" H 6100 2928 50  0000 C CNN
 F 1 "PCF8574" H 6100 2837 50  0000 C CNN
-F 2 "Housings_DIP:DIP-16_W7.62mm_LongPads" H 6100 2050 50  0001 C CNN
+F 2 "" H 6100 2050 50  0001 C CNN
 F 3 "http://www.nxp.com/documents/data_sheet/PCF8574_PCF8574A.pdf" H 6100 2050 50  0001 C CNN
 	1    6100 2050
@@
 	-1   0    0    1
 $EndComp
+$Comp
+L DC-DC_MP2307:DC-DC_BuckModule U2
+U 1 1 5C13D8E2
+P 9750 1500
+F 0 "U2" H 9750 1801 39  0000 C CNN
+F 1 "DC-DC_BuckModule" H 9750 1726 39  0000 C CNN
+F 2 "" H 9750 1500 39  0001 C CNN
+F 3 "" H 9750 1500 39  0001 C CNN
+	1    9750 1500
+	1    0    0    -1
+$EndComp
 Wire Wire Line
 	10050 1400 10150 1400
@@
 F 0 "JP1" H 9300 2535 50  0000 C CNN
 F 1 "Jumper_NO_Small" H 9300 2444 50  0000 C CNN
-F 2 "Jumper:SolderJumper-3_P1.3mm_Open_Pad1.0x1.5mm" H 9300 2350 50  0001 C CNN
+F 2 "" H 9300 2350 50  0001 C CNN
 F 3 "~" H 9300 2350 50  0001 C CNN
 	1    9300 2350
@@
 F 0 "SW3" H 7750 2735 50  0000 C CNN
 F 1 "SW_DPDT_x2" H 7750 2644 50  0000 C CNN
-F 2 "Buttons_Switches_THT:SW_CuK_JS202011CQN_DPDT_Straight" H 7750 2450 50  0001 C CNN
+F 2 "" H 7750 2450 50  0001 C CNN
 F 3 "" H 7750 2450 50  0001 C CNN
 	2    7750 2450
@@
 F 0 "SW3" H 7800 1585 50  0000 C CNN
 F 1 "SW_DPDT_x2" H 7800 1494 50  0000 C CNN
-F 2 "Buttons_Switches_THT:SW_CuK_JS202011CQN_DPDT_Straight" H 7800 1300 50  0001 C CNN
+F 2 "" H 7800 1300 50  0001 C CNN
 F 3 "" H 7800 1300 50  0001 C CNN
 	1    7800 1300
 	1    0    0    -1
 $EndComp
+Wire Wire Line
+	9450 1400 8000 1400
 NoConn ~ 7950 2350
 Text GLabel 7350 1150 1    50   Input ~ 0
@@
 Wire Wire Line
 	6650 5200 6700 5200
-Wire Wire Line
-	9450 1400 8000 1400
-$Comp
-L DC-DC_MP2307:DC-DC_BuckModule U2
-U 1 1 5C1765C0
-P 9750 1500
-F 0 "U2" H 9750 1801 39  0000 C CNN
-F 1 "DC-DC_BuckModule" H 9750 1726 39  0000 C CNN
-F 2 "Placa:DC-DC-MP2307" H 9750 1500 39  0001 C CNN
-F 3 "" H 9750 1500 39  0001 C CNN
-	1    9750 1500
-	1    0    0    -1
-$EndComp
 $EndSCHEMATC
