File: Robot_Veloz-master/Robot_Veloz/Robot_Veloz/Hardware/Placa/Placa/Placa.sch (KiCad schematic (older format))
At the start: 39 parts, among them J1 Conn_01x03, J10 Conn_01x03, J11 Conn_01x03, J12 Conn_01x03, J13 Conn_01x02, J14 Conn_01x02, J15 Conn_01x08, J16 Conn_01x08, J2 Conn_01x03, J3 Conn_01x03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

Commit message: esquema placa terminado
Parts:
- removed A1: Arduino_Nano_v3.x, Module:Arduino_Nano, symbol MCU_Module:Arduino_Nano_v3.x
- removed C1, C2: C, Capacitor_SMD:C_0805_2012Metric_Pad1.15x1.40mm_HandSolder, symbol Device:C
- removed D5, D6: NeoPixel_THT, LED_THT:LED_D5.0mm-4_RGB, symbol LED:NeoPixel_THT
- removed J10, J11, J12: Conn_01x03, Connector_PinHeader_2.54mm:PinHeader_1x06_P2.54mm_Vertical, symbol Connector_Generic:Conn_01x03
- removed J13, J14: Conn_01x02, Connector_PinHeader_2.54mm:PinHeader_1x06_P2.54mm_Vertical, symbol Connector_Generic:Conn_01x02
- removed J15, J16: Conn_01x08, Connector_PinHeader_2.54mm:PinHeader_1x06_P2.54mm_Vertical, symbol Connector_Generic:Conn_01x08
- removed JP1: Jumper_NO_Small, symbol Device:Jumper_NO_Small
- removed R7, R8: R_Small, Resistor_SMD:R_0805_2012Metric_Pad1.15x1.40mm_HandSolder, symbol Device:R_Small
- removed SW3: SW_DPDT_x2, symbol Switch:SW_DPDT_x2
- removed U1: PCF8574, symbol Interface_Expansion:PCF8574
- removed U2: DC-DC_BuckModule, symbol DC-DC_MP2307:DC-DC_BuckModule
- D?: renamed from D1; footprint LED_THT:LED_D3.0mm -> (none)
- D?: renamed from D3; footprint LED_THT:LED_D3.0mm -> (none)
- D?: renamed from D4; footprint Diode_THT:D_DO-41_SOD81_P7.62mm_Horizontal -> (none)
- D?: renamed from D2; footprint Diode_THT:D_DO-41_SOD81_P7.62mm_Horizontal -> (none)
- J?: renamed from J3; footprint Connector_JST:JST_XH_B03B-XH-A_1x03_P2.50mm_Vertical -> (none)
- J?: renamed from J6; footprint Connector_JST:JST_XH_B03B-XH-A_1x03_P2.50mm_Vertical -> (none)
- J?: renamed from J7; footprint Connector_JST:JST_XH_B03B-XH-A_1x03_P2.50mm_Vertical -> (none)
- J?: renamed from J1; footprint Connector_PinHeader_2.54mm:PinHeader_1x06_P2.54mm_Vertical -> (none)
- J?: renamed from J2; footprint Connector_PinHeader_2.54mm:PinHeader_1x06_P2.54mm_Vertical -> (none)
- J?: renamed from J4; footprint Connector_PinHeader_2.54mm:PinHeader_1x06_P2.54mm_Vertical -> (none)
- J?: renamed from J5; footprint Connector_PinHeader_2.54mm:PinHeader_1x06_P2.54mm_Vertical -> (none)
- J?: renamed from J8; footprint Connector_PinHeader_2.54mm:PinHeader_1x06_P2.54mm_Vertical -> (none)
- J?: renamed from J9; footprint Connector_PinHeader_2.54mm:PinHeader_1x06_P2.54mm_Vertical -> (none)
- R?: renamed from R1; footprint Resistor_SMD:R_0805_2012Metric_Pad1.15x1.40mm_HandSolder -> (none)
- R?: renamed from R2; footprint Resistor_SMD:R_0805_2012Metric_Pad1.15x1.40mm_HandSolder -> (none)
- R?: renamed from R3; footprint Resistor_SMD:R_0805_2012Metric_Pad1.15x1.40mm_HandSolder -> (none)
- R?: renamed from R6; footprint Resistor_SMD:R_0805_2012Metric_Pad1.15x1.40mm_HandSolder -> (none)
- R?: renamed from R4; footprint Resistor_SMD:R_0805_2012Metric_Pad1.15x1.40mm_HandSolder -> (none)
- R?: renamed from R5; footprint Resistor_SMD:R_0805_2012Metric_Pad1.15x1.40mm_HandSolder -> (none)
- renumbered SW1 to SW?, SW2 to SW?
Connections:
- net +5V: no longer J?.1 (Pin_1)
- net GND: no longer J?.2 (Pin_2)
- net LINEA_1: no longer names the net of J?.3 (Pin_3)
- net LINEA_2: no longer names the net of J?.4 (Pin_4)
- net LINEA_3: no longer names the net of J?.5 (Pin_5)
- net LINEA_SEL: no longer names the net of J?.6 (Pin_6)
- no-connect marks 11 -> 3
Other:
- moved on the sheet: J?
